File: schematics/extboard.sch (EAGLE design)
At the start: 37 parts, among them X1 FPS009-3000

Commit message: schematics: board rev. A
Parts:
- removed C11, C12, C13, C14: (no value), rcl:CPOL-EUE2.5-7
- removed C3, C4, C5, C6, C7, C8: (no value), rcl:C-EU050-035X075
- removed R1: 100k, rcl:R-EU_0207/10
- removed R10, R11, R12, R13, R14, R15, R16, R17, R18, R19, R20, R8, R9: (no value), rcl:R-EU_0207/10
- removed X1: FPS009-3000, con-yamaichi:FPS009-3000
- added C15, C16: 0u1, rcl:C-EU050-035X075
- added C18: 2u2, rcl:CPOL-EUE2.5-7
- added R21: 250, rcl:R-EU_0207/10
- added R22: 10, rcl:R-EU_0207/10
- added SV2, SV3: (no value), con-lstb:MA03-1
- added U$2: LTC1257, ltc1257:LTC1257
- added X2: 1503_02, con-lumberg:1503_02
- added X3: SDBMF, farnell-sd:SDBMF
- C10: value (none) -> 2u2
- R2: value 1k -> 250
- R3: value (none) -> 10
- R6, R7: value (none) -> 10k
Connections:
- new net N$16: R7.1, SV2.3
- new net N$17: SV2.2, U$1.D_OUT
- new net N$18: SV3.2, X2.1
- new net N$19: R6.2, U$2.D_OUT
- new net N$21: C16.1, R21.2, SV3.3
- new net N$22: R21.1, U$2.V_OUT
- new net N$23: C18.-, R22.2
- net GND: now also C15.2, C16.2, R22.1, R4.2, R5.2, R6.1, R7.2, U$2.GND, X2.2, X3.3, X3.6; no longer R1.1, X1.3, X1.6
- net N$1: now also U$2.CLK
- net N$10: now also R4.1, X3.9; no longer R4.2, X1.9
- net N$11: now also X3.4; no longer R4.1, R5.1, X1.4
- net N$12: now also X3.1; no longer X1.1
- net N$13: now also X3.2; no longer X1.2
- net N$14: now also X3.5; no longer X1.5
- net N$15: now also X3.7; no longer X1.7
- net N$3: now also U$2.~LOAD
- net N$4: now also SV2.1, U$2.D_IN; no longer R1.2, U$1.D_OUT
- net N$6: now also C15.1, C18.+, U$2.REF
- net N$7: now also SV3.1, X2.3
- net N$9: now also R5.1, X3.8; no longer R5.2, X1.8
- net VCC: now also U$2.V_CC
Other:
- moved on the sheet: C9, R2, R4, R5, R6, R7

Commit message: schematics: Fix in Rev A
Parts:
- added C1B: 2u2, rcl:CPOL-EUE2.5-7
- renumbered C1 to C3A, C10 to C2A, C15 to C3B, C16 to C4B, C18 to C2B, C2 to C4A, C9 to C1A, R2 to R1A, R21 to R1B, R22 to R2B, R3 to R2A, R6 to R3B, R7 to R3A, SV1 to X3-BRD, SV2 to J1, SV3 to J2, U$1 to U1, U$2 to U2, X2 to X2-JACK, X3 to X1-SD
Connections:
- net GND: now also C1B.-; no longer R4.2, R5.2
- net N$11: now also C1B.+, R4.2, R5.2

Commit message: schematics: next iteration
Connections:
- new net N$24: X1-SD.SW1, X3-BRD.34
- new net N$25: X1-SD.SW2, X3-BRD.36
- new net N$26: X1-SD.SW3, X3-BRD.38
Other:
- moved on the sheet: C1B, R4, R5, X1-SD
Changed lines of the file:
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@@
 <sheet>
 <plain>
-<rectangle x1="-17.78" y1="17.78" x2="-10.16" y2="63.5" layer="91"/>
-<rectangle x1="-10.16" y1="17.78" x2="-2.54" y2="43.18" layer="91"/>
 </plain>
 <instances>
@@
 <instance part="R1A" gate="G$1" x="73.66" y="17.78"/>
 <instance part="R2A" gate="G$1" x="104.14" y="7.62" rot="R90"/>
-<instance part="R4" gate="G$1" x="-20.32" y="88.9"/>
-<instance part="R5" gate="G$1" x="-20.32" y="91.44"/>
+<instance part="R4" gate="G$1" x="96.52" y="73.66" rot="R180"/>
+<instance part="R5" gate="G$1" x="86.36" y="71.12" rot="R180"/>
 <instance part="R3A" gate="G$1" x="12.7" y="22.86" rot="R90"/>
 <instance part="GND2" gate="1" x="63.5" y="7.62"/>
-<instance part="GND3" gate="1" x="25.4" y="58.42"/>
+<instance part="GND3" gate="1" x="25.4" y="40.64"/>
 <instance part="GND4" gate="1" x="81.28" y="-5.08"/>
 <instance part="GND9" gate="1" x="-5.08" y="-15.24"/>
@@
 <instance part="J2" gate="G$1" x="114.3" y="33.02" rot="R270"/>
 <instance part="X2-JACK" gate="G$1" x="149.86" y="17.78"/>
-<instance part="X1-SD" gate="G$1" x="-33.02" y="91.44"/>
-<instance part="C1B" gate="G$1" x="25.4" y="86.36"/>
+<instance part="X1-SD" gate="G$1" x="109.22" y="71.12" rot="R180"/>
+<instance part="C1B" gate="G$1" x="33.02" y="73.66" rot="R270"/>
 </instances>
 <busses>
@@
 </segment>
 <segment>
+<pinref part="C1B" gate="G$1" pin="-"/>
 <pinref part="GND3" gate="1" pin="GND"/>
-<wire x1="25.4" y1="60.96" x2="25.4" y2="66.04" width="0.1524" layer="91"/>
+<wire x1="25.4" y1="43.18" x2="25.4" y2="66.04" width="0.1524" layer="91"/>
 <pinref part="X3-BRD" gate="1" pin="39"/>
-<wire x1="-2.54" y1="66.04" x2="2.54" y2="66.04" width="0.1524" layer="91"/>
-<wire x1="2.54" y1="66.04" x2="25.4" y2="66.04" width="0.1524" layer="91"/>
+<wire x1="25.4" y1="66.04" x2="25.4" y2="73.66" width="0.1524" layer="91"/>
+<wire x1="25.4" y1="73.66" x2="27.94" y2="73.66" width="0.1524" layer="91"/>
 <pinref part="X1-SD" gate="G$1" pin="3"/>
-<wire x1="2.54" y1="96.52" x2="2.54" y2="104.14" width="0.1524" layer="91"/>
-<wire x1="2.54" y1="104.14" x2="-27.94" y2="104.14" width="0.1524" layer="91"/>
+<wire x1="40.64" y1="66.04" x2="40.64" y2="58.42" width="0.1524" layer="91"/>
+<wire x1="40.64" y1="58.42" x2="104.14" y2="58.42" width="0.1524" layer="91"/>
 <pinref part="X1-SD" gate="G$1" pin="6"/>
-<wire x1="-27.94" y1="96.52" x2="2.54" y2="96.52" width="0.1524" layer="91"/>
-<junction x="2.54" y="96.52"/>
-<wire x1="2.54" y1="96.52" x2="2.54" y2="66.04" width="0.1524" layer="91"/>
-<junction x="2.54" y="66.04"/>
-<pinref part="C1B" gate="G$1" pin="-"/>
-<wire x1="25.4" y1="81.28" x2="25.4" y2="66.04" width="0.1524" layer="91"/>
+<wire x1="104.14" y1="66.04" x2="40.64" y2="66.04" width="0.1524" layer="91"/>
+<junction x="40.64" y="66.04"/>
+<wire x1="40.64" y1="66.04" x2="-2.54" y2="66.04" width="0.1524" layer="91"/>
+<wire x1="40.64" y1="66.04" x2="25.4" y2="66.04" width="0.1524" layer="91"/>
 <junction x="25.4" y="66.04"/>
 </segment>
@@
 <segment>
 <pinref part="X3-BRD" gate="1" pin="29"/>
-<wire x1="-2.54" y1="53.34" x2="12.7" y2="53.34" width="0.1524" layer="91"/>
-<wire x1="12.7" y1="53.34" x2="12.7" y2="109.22" width="0.1524" layer="91"/>
+<wire x1="-2.54" y1="53.34" x2="104.14" y2="53.34" width="0.1524" layer="91"/>
 <pinref part="X1-SD" gate="G$1" pin="1"/>
-<wire x1="-27.94" y1="109.22" x2="12.7" y2="109.22" width="0.1524" layer="91"/>
 </segment>
 </net>
@@
 <segment>
 <pinref part="X3-BRD" gate="1" pin="27"/>
-<wire x1="-2.54" y1="50.8" x2="10.16" y2="50.8" width="0.1524" layer="91"/>
-<wire x1="10.16" y1="50.8" x2="10.16" y2="106.68" width="0.1524" layer="91"/>
+<wire x1="-2.54" y1="50.8" x2="101.6" y2="50.8" width="0.1524" layer="91"/>
 <pinref part="X1-SD" gate="G$1" pin="2"/>
-<wire x1="-27.94" y1="106.68" x2="10.16" y2="106.68" width="0.1524" layer="91"/>
+<wire x1="104.14" y1="55.88" x2="101.6" y2="55.88" width="0.1524" layer="91"/>
+<wire x1="101.6" y1="55.88" x2="101.6" y2="50.8" width="0.1524" layer="91"/>
 </segment>
 </net>
@@
 <segment>
 <pinref part="X3-BRD" gate="1" pin="25"/>
-<wire x1="-2.54" y1="48.26" x2="7.62" y2="48.26" width="0.1524" layer="91"/>
-<wire x1="7.62" y1="48.26" x2="7.62" y2="99.06" width="0.1524" layer="91"/>
+<wire x1="-2.54" y1="48.26" x2="99.06" y2="48.26" width="0.1524" layer="91"/>
 <pinref part="X1-SD" gate="G$1" pin="5"/>
-<wire x1="-27.94" y1="99.06" x2="7.62" y2="99.06" width="0.1524" layer="91"/>
+<wire x1="104.14" y1="63.5" x2="99.06" y2="63.5" width="0.1524" layer="91"/>
+<wire x1="99.06" y1="63.5" x2="99.06" y2="48.26" width="0.1524" layer="91"/>
 </segment>
 </net>
@@
 <segment>
 <pinref part="X3-BRD" gate="1" pin="23"/>
-<wire x1="-2.54" y1="45.72" x2="5.08" y2="45.72" width="0.1524" layer="91"/>
-<wire x1="5.08" y1="45.72" x2="5.08" y2="93.98" width="0.1524" layer="91"/>
+<wire x1="-2.54" y1="45.72" x2="7.62" y2="45.72" width="0.1524" layer="91"/>
+<wire x1="7.62" y1="45.72" x2="7.62" y2="68.58" width="0.1524" layer="91"/>
 <pinref part="X1-SD" gate="G$1" pin="7"/>
-<wire x1="5.08" y1="93.98" x2="-27.94" y2="93.98" width="0.1524" layer="91"/>
+<wire x1="7.62" y1="68.58" x2="104.14" y2="68.58" width="0.1524" layer="91"/>
 </segment>
 </net>
@@
 <pinref part="X1-SD" gate="G$1" pin="8"/>
 <pinref part="R5" gate="G$1" pin="1"/>
-<wire x1="-27.94" y1="91.44" x2="-25.4" y2="91.44" width="0.1524" layer="91"/>
+<wire x1="104.14" y1="71.12" x2="91.44" y2="71.12" width="0.1524" layer="91"/>
 </segment>
 </net>
@@
 <pinref part="X1-SD" gate="G$1" pin="9"/>
 <pinref part="R4" gate="G$1" pin="1"/>
-<wire x1="-27.94" y1="88.9" x2="-25.4" y2="88.9" width="0.1524" layer="91"/>
+<wire x1="104.14" y1="73.66" x2="101.6" y2="73.66" width="0.1524" layer="91"/>
 </segment>
 </net>
 <net name="N$11" class="0">
 <segment>
+<pinref part="R5" gate="G$1" pin="2"/>
+<pinref part="C1B" gate="G$1" pin="+"/>
+<wire x1="38.1" y1="73.66" x2="35.56" y2="73.66" width="0.1524" layer="91"/>
 <pinref part="X3-BRD" gate="1" pin="37"/>
-<wire x1="-2.54" y1="63.5" x2="0" y2="63.5" width="0.1524" layer="91"/>
+<wire x1="50.8" y1="63.5" x2="38.1" y2="63.5" width="0.1524" layer="91"/>
+<wire x1="38.1" y1="63.5" x2="-2.54" y2="63.5" width="0.1524" layer="91"/>
+<wire x1="38.1" y1="73.66" x2="38.1" y2="63.5" width="0.1524" layer="91"/>
+<junction x="38.1" y="63.5"/>
+<wire x1="50.8" y1="63.5" x2="50.8" y2="60.96" width="0.1524" layer="91"/>
 <pinref part="X1-SD" gate="G$1" pin="4"/>
-<wire x1="-27.94" y1="101.6" x2="0" y2="101.6" width="0.1524" layer="91"/>
-<wire x1="0" y1="101.6" x2="0" y2="91.44" width="0.1524" layer="91"/>
-<pinref part="R5" gate="G$1" pin="2"/>
-<wire x1="0" y1="91.44" x2="0" y2="88.9" width="0.1524" layer="91"/>
-<wire x1="0" y1="88.9" x2="0" y2="63.5" width="0.1524" layer="91"/>
-<wire x1="-15.24" y1="91.44" x2="0" y2="91.44" width="0.1524" layer="91"/>
-<junction x="0" y="91.44"/>
+<wire x1="104.14" y1="60.96" x2="50.8" y2="60.96" width="0.1524" layer="91"/>
+<wire x1="50.8" y1="63.5" x2="50.8" y2="71.12" width="0.1524" layer="91"/>
+<junction x="50.8" y="63.5"/>
+<wire x1="81.28" y1="71.12" x2="50.8" y2="71.12" width="0.1524" layer="91"/>
+<wire x1="50.8" y1="71.12" x2="50.8" y2="73.66" width="0.1524" layer="91"/>
+<junction x="50.8" y="71.12"/>
 <pinref part="R4" gate="G$1" pin="2"/>
-<wire x1="0" y1="88.9" x2="-15.24" y2="88.9" width="0.1524" layer="91"/>
-<junction x="0" y="88.9"/>
-<pinref part="C1B" gate="G$1" pin="+"/>
-<wire x1="0" y1="101.6" x2="25.4" y2="101.6" width="0.1524" layer="91"/>
-<wire x1="25.4" y1="101.6" x2="25.4" y2="88.9" width="0.1524" layer="91"/>
-<junction x="0" y="101.6"/>
-</segment>
-</net>
+<wire x1="50.8" y1="73.66" x2="91.44" y2="73.66" width="0.1524" layer="91"/>
+</segment>
+</net>
+<net name="N$24" class="0">
+<segment>
+<pinref part="X1-SD" gate="G$1" pin="SW1"/>
+<wire x1="-27.94" y1="78.74" x2="104.14" y2="78.74" width="0.1524" layer="91"/>
+<pinref part="X3-BRD" gate="1" pin="34"/>
+<wire x1="-17.78" y1="58.42" x2="-27.94" y2="58.42" width="0.1524" layer="91"/>
+<wire x1="-27.94" y1="58.42" x2="-27.94" y2="78.74" width="0.1524" layer="91"/>
+</segment>
+</net>
+<net name="N$25" class="0">
+<segment>
+<pinref part="X1-SD" gate="G$1" pin="SW2"/>
+<wire x1="104.14" y1="81.28" x2="-25.4" y2="81.28" width="0.1524" layer="91"/>
+<wire x1="-25.4" y1="81.28" x2="-25.4" y2="60.96" width="0.1524" layer="91"/>
+<pinref part="X3-BRD" gate="1" pin="36"/>
+<wire x1="-25.4" y1="60.96" x2="-17.78" y2="60.96" width="0.1524" layer="91"/>
+</segment>
+</net>
+<net name="N$26" class="0">
+<segment>
+<pinref part="X1-SD" gate="G$1" pin="SW3"/>
+<wire x1="-22.86" y1="83.82" x2="104.14" y2="83.82" width="0.1524" layer="91"/>
+<wire x1="-22.86" y1="83.82" x2="-22.86" y2="63.5" width="0.1524" layer="91"/>
+<pinref part="X3-BRD" gate="1" pin="38"/>
+<wire x1="-22.86" y1="63.5" x2="-17.78" y2="63.5" width="0.1524" layer="91"/>
+</segment>
+</net>
